Commit message: Fixed pointcloud rgbd_frame issue

File: udacity_bot/urdf/race_car.xacro (robot description, xacro)
@@ -215,4 +215,14 @@
     <dynamics damping="1.0" friction="1.0"/>
   </joint>
+  <joint name="camera_rgbd_joint" type="fixed">
+    <!-- these values have to be these values otherwise the gazebo camera
+        image won't be aligned properly with the frame it is supposedly
+        originating from -->
+    <origin xyz="0 0 0" rpy="${-pi/2} 0 ${-pi/2}"/>
+    <parent link="camera"/>
+    <child link="camera_rgbd_frame"/>
+  </joint>
+  <link name="camera_rgbd_frame">
+  </link>
   <link name="hokuyo">
     <inertial>
